File: Schematic/4760_Final.sch (KiCad schematic (older format))
At the start: 10 parts

Commit message: init commit, massive repo for 4760 Final Project
Parts:
- removed F?: 10A, symbol Device:Fuse
Connections:
- net HOT_AC: now also SW?.1 (A)
- net at K?.7, K?.8: now also J?.2 (Pin_2), J?.2 (Pin_2); no longer SW?.1 (A)
- net at U?.1 (IP+): now also SW?.2 (B)
- net GNDPWR renamed GFCI
Other:
- moved on the sheet: K?, Q?, R?, SW?, U?
Changed lines of the file:
@@
 Comment4 ""
 $EndDescr
-Text GLabel 2000 4300 2    50   Input ~ 0
+Text GLabel 2050 4450 0    50   Input ~ 0
 HOT_AC
 $Comp
 L Relay:DIPxx-1Axx-12x K?
 U 1 1 5D9D0B46
-P 3900 3650
-F 0 "K?" V 3333 3650 50  0000 C CNN
-F 1 "RENAME LATER" V 3424 3650 50  0000 C CNN
-F 2 "Relay_THT:Relay_StandexMeder_DIP_LowProfile" H 4250 3600 50  0001 L CNN
-F 3 "https://standexelectronics.com/wp-content/uploads/datasheet_reed_relay_DIP.pdf" H 3900 3650 50  0001 C CNN
-	1    3900 3650
+P 4350 3800
+F 0 "K?" V 3783 3800 50  0000 C CNN
+F 1 "RENAME LATER" V 3874 3800 50  0000 C CNN
+F 2 "Relay_THT:Relay_StandexMeder_DIP_LowProfile" H 4700 3750 50  0001 L CNN
+F 3 "https://standexelectronics.com/wp-content/uploads/datasheet_reed_relay_DIP.pdf" H 4350 3800 50  0001 C CNN
+	1    4350 3800
 	0    1    1    0
 $EndComp
@@
 L Sensor_Current:ACS711xEXLT-15AB U?
 U 1 1 5D9EAF0B
-P 2750 3450
-F 0 "U?" V 2796 3893 50  0000 L CNN
-F 1 "NAME LATER" V 2705 3893 50  0000 L CNN
-F 2 "Sensor_Current:Allegro_QFN-12-10-1EP_3x3mm_P0.5mm" H 3100 3400 50  0001 L CIN
-F 3 "http://www.allegromicro.com/~/Media/Files/Datasheets/ACS711-Datasheet.ashx" H 2750 3450 50  0001 C CNN
-	1    2750 3450
+P 3200 3600
+F 0 "U?" V 3246 4043 50  0000 L CNN
+F 1 "NAME LATER" V 3155 4043 50  0000 L CNN
+F 2 "Sensor_Current:Allegro_QFN-12-10-1EP_3x3mm_P0.5mm" H 3550 3550 50  0001 L CIN
+F 3 "http://www.allegromicro.com/~/Media/Files/Datasheets/ACS711-Datasheet.ashx" H 3200 3600 50  0001 C CNN
+	1    3200 3600
 	0    -1   -1   0
 $EndComp
 Wire Wire Line
-	2200 3850 2200 4150
-Wire Wire Line
-	2850 3850 2850 4600
-Wire Wire Line
-	2850 4600 2700 4600
-Connection ~ 2850 3850
-Wire Wire Line
-	2700 4600 2700 5350
+	2650 4000 2650 4300
 Wire Wire Line
 	2700 5350 2900 5350
-$Comp
-L Device:Fuse F?
-U 1 1 5DA0E26C
-P 1950 4150
-F 0 "F?" V 1753 4150 50  0000 C CNN
-F 1 "10A" V 1844 4150 50  0000 C CNN
-F 2 "" V 1880 4150 50  0001 C CNN
-F 3 "~" H 1950 4150 50  0001 C CNN
-	1    1950 4150
-	0    1    1    0
-$EndComp
-Wire Wire Line
-	2100 4150 2200 4150
+Wire Wire Line
+	2550 4300 2650 4300
 Text Notes 3500 -350 0    50   ~ 0
 third prong???\n
 Text Notes 5700 -650 0    50   ~ 0
 PIC32 schematic symbol. bring that in
-Text GLabel 1500 3800 2    50   Input ~ 0
+Text GLabel 1500 3950 2    50   Input ~ 0
 NEUTRAL
 Wire Wire Line
-	2850 3850 3600 3850
+	3300 4000 3600 4000
 $Comp
 L power:NEUT #PWR?
@@
 	1500 4050 1350 4050
 Wire Wire Line
-	1350 4150 1800 4150
-Wire Wire Line
-	1800 4150 1800 4300
-Connection ~ 1800 4150
+	2150 4300 2150 4450
 Wire Wire Line
 	1350 4250 1350 4400
@@
 Wire Wire Line
 	1350 4400 1450 4400
-$Comp
-L power:GNDPWR #PWR?
-U 1 1 5DA62B98
-P 1350 4650
-F 0 "#PWR?" H 1350 4450 50  0001 C CNN
-F 1 "GNDPWR" H 1354 4496 50  0000 C CNN
-F 2 "" H 1350 4600 50  0001 C CNN
-F 3 "" H 1350 4600 50  0001 C CNN
-	1    1350 4650
-	1    0    0    -1
-$EndComp
-Wire Wire Line
-	1350 4400 1350 4650
-Connection ~ 1350 4400
-Wire Wire Line
-	2000 4300 1800 4300
 $Comp
 L Connector:Conn_01x03_Female J?
@@
 	1500 3700 1500 4050
 Wire Wire Line
-	5950 3850 5950 4000
-Wire Wire Line
 	6700 4300 7600 4300
 Wire Wire Line
@@
 	7350 4400 7600 4400
 Wire Wire Line
-	3150 3450 3300 3450
-Wire Wire Line
-	2350 3450 2350 3200
+	3600 3600 3750 3600
+Wire Wire Line
+	2800 3600 2800 3350
 $Comp
 L power:+5V #PWR?
 U 1 1 5DC04101
-P 2350 3200
-F 0 "#PWR?" H 2350 3050 50  0001 C CNN
-F 1 "+5V" H 2365 3373 50  0000 C CNN
-F 2 "" H 2350 3200 50  0001 C CNN
-F 3 "" H 2350 3200 50  0001 C CNN
-	1    2350 3200
+P 2800 3350
+F 0 "#PWR?" H 2800 3200 50  0001 C CNN
+F 1 "+5V" H 2815 3523 50  0000 C CNN
+F 2 "" H 2800 3350 50  0001 C CNN
+F 3 "" H 2800 3350 50  0001 C CNN
+	1    2800 3350
 	1    0    0    -1
 $EndComp
@@
 L power:GND #PWR?
 U 1 1 5DC0463E
-P 3300 3500
-F 0 "#PWR?" H 3300 3250 50  0001 C CNN
-F 1 "GND" H 3305 3327 50  0000 C CNN
-F 2 "" H 3300 3500 50  0001 C CNN
-F 3 "" H 3300 3500 50  0001 C CNN
-	1    3300 3500
-	1    0    0    -1
-$EndComp
-Wire Wire Line
-	3300 3500 3300 3450
-Text Label 2750 2600 0    50   ~ 0
+P 3750 3650
+F 0 "#PWR?" H 3750 3400 50  0001 C CNN
+F 1 "GND" H 3755 3477 50  0000 C CNN
+F 2 "" H 3750 3650 50  0001 C CNN
+F 3 "" H 3750 3650 50  0001 C CNN
+	1    3750 3650
+	1    0    0    -1
+$EndComp
+Wire Wire Line
+	3750 3650 3750 3600
+Text Label 3200 2750 0    50   ~ 0
 CURRENT_BEFORE_RELAY
 Wire Wire Line
-	2750 2600 2750 3050
-NoConn ~ 3150 3250
-NoConn ~ 3150 3350
-NoConn ~ 3150 3550
-NoConn ~ 3150 3650
-Wire Wire Line
-	2850 3050 2850 2800
-Wire Wire Line
-	2850 2800 2900 2800
-Text Label 2900 2800 0    50   ~ 0
+	3200 2750 3200 3200
+NoConn ~ 3600 3400
+NoConn ~ 3600 3500
+NoConn ~ 3600 3700
+NoConn ~ 3600 3800
+Wire Wire Line
+	3300 3200 3300 2950
+Wire Wire Line
+	3300 2950 3350 2950
+Text Label 3350 2950 0    50   ~ 0
 ~FAULT_BEFORE_RELAY
 Wire Wire Line
-	3600 3450 3600 2950
-Wire Wire Line
-	4200 3450 4200 3000
-Wire Wire Line
-	6100 4000 5950 4000
-Wire Wire Line
-	6500 4000 6700 4000
+	4050 3600 4050 3100
+Wire Wire Line
+	4650 3600 4650 3150
 Wire Wire Line
 	6700 4000 6700 3850
@@
 	6700 4000 6700 4300
 Connection ~ 6700 4000
-Text Label 4800 5300 2    50   ~ 0
+Text Label 5450 5750 2    50   ~ 0
 ~ENABLE_PIC
 $Comp
 L 4760_Final-rescue:NMOS-cuauv Q?
 U 1 1 5DC24080
-P 5200 5300
-F 0 "Q?" H 5390 5346 50  0000 L CNN
-F 1 "NMOS" H 5390 5255 50  0000 L CNN
-F 2 "cuauv:SOT-23-3" H 5400 5400 50  0001 C CNN
-F 3 "" H 5500 5350 50  0000 C CNN
-	1    5200 5300
-	1    0    0    -1
-$EndComp
-Wire Wire Line
-	4800 5300 5000 5300
+P 5850 5750
+F 0 "Q?" H 6040 5796 50  0000 L CNN
+F 1 "NMOS" H 6040 5705 50  0000 L CNN
+F 2 "cuauv:SOT-23-3" H 6050 5850 50  0001 C CNN
+F 3 "" H 6150 5800 50  0000 C CNN
+	1    5850 5750
+	1    0    0    -1
+$EndComp
+Wire Wire Line
+	5450 5750 5650 5750
 $Comp
 L power:+5V #PWR?
 U 1 1 5DC27787
-P 5300 4500
-F 0 "#PWR?" H 5300 4350 50  0001 C CNN
-F 1 "+5V" H 5315 4673 50  0000 C CNN
-F 2 "" H 5300 4500 50  0001 C CNN
-F 3 "" H 5300 4500 50  0001 C CNN
-	1    5300 4500
-	1    0    0    -1
-$EndComp
-Wire Wire Line
-	5300 5500 5300 5650
+P 5950 4950
+F 0 "#PWR?" H 5950 4800 50  0001 C CNN
+F 1 "+5V" H 5965 5123 50  0000 C CNN
+F 2 "" H 5950 4950 50  0001 C CNN
+F 3 "" H 5950 4950 50  0001 C CNN
+	1    5950 4950
+	1    0    0    -1
+$EndComp
+Wire Wire Line
+	5950 5950 5950 6100
 $Comp
 L power:GND #PWR?
 U 1 1 5DC28C9F
-P 5300 5650
-F 0 "#PWR?" H 5300 5400 50  0001 C CNN
-F 1 "GND" H 5305 5477 50  0000 C CNN
-F 2 "" H 5300 5650 50  0001 C CNN
-F 3 "" H 5300 5650 50  0001 C CNN
-	1    5300 5650
-	1    0    0    -1
-$EndComp
-Text Label 3600 2950 0    50   ~ 0
+P 5950 6100
+F 0 "#PWR?" H 5950 5850 50  0001 C CNN
+F 1 "GND" H 5955 5927 50  0000 C CNN
+F 2 "" H 5950 6100 50  0001 C CNN
+F 3 "" H 5950 6100 50  0001 C CNN
+	1    5950 6100
+	1    0    0    -1
+$EndComp
+Text Label 4050 3100 0    50   ~ 0
 ENABLE_RELAY
 $Comp
 L power:GND #PWR?
 U 1 1 5DC2962E
-P 4300 3000
-F 0 "#PWR?" H 4300 2750 50  0001 C CNN
-F 1 "GND" H 4400 3100 50  0000 R CNN
-F 2 "" H 4300 3000 50  0001 C CNN
-F 3 "" H 4300 3000 50  0001 C CNN
-	1    4300 3000
-	1    0    0    -1
-$EndComp
-Wire Wire Line
-	4300 3000 4200 3000
-Wire Wire Line
-	2550 3850 2200 3850
-Wire Wire Line
-	4200 3850 5950 3850
+P 4750 3150
+F 0 "#PWR?" H 4750 2900 50  0001 C CNN
+F 1 "GND" H 4850 3250 50  0000 R CNN
+F 2 "" H 4750 3150 50  0001 C CNN
+F 3 "" H 4750 3150 50  0001 C CNN
+	1    4750 3150
+	1    0    0    -1
+$EndComp
+Wire Wire Line
+	4750 3150 4650 3150
+Wire Wire Line
+	3000 4000 2650 4000
 $Comp
 L Switch:SW_SPST SW?
 U 1 1 5DC1C446
-P 6300 4000
-F 0 "SW?" H 6300 4235 50  0000 C CNN
-F 1 "SW_SPST" H 6300 4144 50  0000 C CNN
-F 2 "" H 6300 4000 50  0001 C CNN
-F 3 "~" H 6300 4000 50  0001 C CNN
-	1    6300 4000
+P 2350 4300
+F 0 "SW?" H 2350 4535 50  0000 C CNN
+F 1 "SW_SPST" H 2350 4444 50  0000 C CNN
+F 2 "" H 2350 4300 50  0001 C CNN
+F 3 "~" H 2350 4300 50  0001 C CNN
+	1    2350 4300
 	1    0    0    -1
 $EndComp
@@
 L Device:R R?
 U 1 1 5DC1D7B2
-P 5300 4850
-F 0 "R?" H 5370 4896 50  0000 L CNN
-F 1 "1k" V 5300 4800 50  0000 L CNN
-F 2 "" V 5230 4850 50  0001 C CNN
-F 3 "~" H 5300 4850 50  0001 C CNN
-	1    5300 4850
-	1    0    0    -1
-$EndComp
-Wire Wire Line
-	5300 5000 5300 5050
-Text Label 5500 5050 0    50   ~ 0
+P 5950 5300
+F 0 "R?" H 6020 5346 50  0000 L CNN
+F 1 "1k" V 5950 5250 50  0000 L CNN
+F 2 "" V 5880 5300 50  0001 C CNN
+F 3 "~" H 5950 5300 50  0001 C CNN
+	1    5950 5300
+	1    0    0    -1
+$EndComp
+Wire Wire Line
+	5950 5450 5950 5500
+Text Label 6150 5500 0    50   ~ 0
 ENABLE_RELAY
 Wire Wire Line
-	5300 5050 5500 5050
-Connection ~ 5300 5050
-Wire Wire Line
-	5300 5050 5300 5100
-Wire Wire Line
-	5300 4500 5300 4700
+	5950 5500 6150 5500
+Connection ~ 5950 5500
+Wire Wire Line
+	5950 5500 5950 5550
+Wire Wire Line
+	5950 4950 5950 5150
 Text Notes 19450 -650 0    118  ~ 0
 Use actual MCU later\n
+Wire Wire Line
+	2050 4450 2150 4450
+Connection ~ 2150 4300
+Wire Wire Line
+	2000 4150 2000 4300
+Wire Wire Line
+	1350 4150 2000 4150
+Wire Wire Line
+	2000 4300 2150 4300
+Wire Wire Line
+	2700 5350 2700 4500
+Wire Wire Line
+	2700 4500 3600 4500
+Wire Wire Line
+	3600 4500 3600 4000
+Connection ~ 3600 4000
+Wire Wire Line
+	3600 4000 4050 4000
+Wire Wire Line
+	4650 4000 6700 4000
 $EndSCHEMATC

Commit message: excluding schematic for Sean Carroll's small pic32 board (which is on the course website), project schematic is finished
Parts:
- removed Q?: NMOS, cuauv:SOT-23-3, symbol 4760_Final-rescue:NMOS-cuauv
- removed U?: RaspberryPi-CM1, symbol MCU_Module:RaspberryPi-CM1
- removed U?: NAME LATER, Sensor_Current:Allegro_QFN-12-10-1EP_3x3mm_P0.5mm, symbol Sensor_Current:ACS711xEXLT-15AB
- added C1: 1nF, symbol Device:C
- added C2: 1uF, symbol Device:C
- added C3: 10uF, symbol Device:CP1
- added D1: RED, symbol Device:LED
- added D2: YELLOW, symbol Device:LED
- added D3: GREEN, symbol Device:LED
- added J?: UART_TTL_TO_USB_CABLE, symbol Connector:Conn_01x03_Female
- added Q1: AOT2618L NMOS, symbol Device:Q_NMOS_DGS
- added R1: 100, symbol Device:R
- added R3, R4: 1.5k, symbol Device:R
- added R5, R6: 1k, symbol Device:R
- added U2: ACHS-7122, symbol 4760_final:ACHS-7122
- J1: renamed from J?; value InputPower -> Supply (Input) Plug
- J2: renamed from J?; value OutputPower -> Client (Output) Sockets
- K1: renamed from K?; value RENAME LATER -> G3NE-210T-US-DC5
- gave numbers to parts that had none: 3
Connections:
- net +5V: now also C2.1, U2.8 (Vdd); no longer R2.1
- net ENABLE_RELAY: now also Q1.1 (D)
- net GND: now also C1.2, C2.2, C3.2, D1.1 (K), D2.1 (K), D3.1 (K), J?.1 (Pin_1), Q1.3 (S), U2.5 (GND)
- net pseudo5VBrick.sch/V_AC: now also U2.3 (Ip-), U2.4 (Ip-)
- net ~ENABLE_PIC: now also Q1.2 (G), R6.1
- net at SW1.2 (B): now also U2.1 (Ip+), U2.2 (Ip+)
- net NEUT renamed NEUTRAL
- new net: C1.1, U2.6 (FLTR)
- new net: D1.2 (A), R3.1
- new net: D2.2 (A), R4.1
- new net: D3.2 (A), R5.1
- new net +5VA: R2.1
- new net I_READING: R1.2, U2.7 (Vout)
- new net I_READING_FLTRED: C3.1, R1.1
- new net PIC32 Sean Caroll Small Board/DIG_OUTPUT_0: R3.2
- new net PIC32 Sean Caroll Small Board/DIG_OUTPUT_1: R4.2
- new net PIC32 Sean Caroll Small Board/DIG_OUTPUT_2: R5.2
- new net PIC32 Sean Caroll Small Board/DIG_OUTPUT_3: R6.2
- new net RX_PIC32: J?.3 (Pin_3)
- new net TX_PIC32: J?.2 (Pin_2)
- no-connect marks 4 -> 0
Other:
- note added: "(RA0)"
- note added: "(RA1)"
- note added: "(RB0)"
- note added: "(RB1)"
- note added: "(RB10)"
- note added: "(RB2)"
- note added: "BLACK"
- note added: "Client HOT AC (red wire)"
- note added: "GFCI \n(green wire)"
- note added: "GREEN (TX Computer)\n"
- note added: "HOT after Current Sensor\n(still black)"
- note added: "Hall Effect Current Sensor\n"
- note added: "Indicator LEDs\n"
- note added: "Inverter \n(Digital Output \n3.3V to 5V buffer)"
- note added: "Neutral\n(white wire)"
- note added: "Outlet Box"
- note added: "PIC32 + Peripherals"
- note added: "RA1"
- note added: "Supply HOT AC \n(black wire)"
- note added: "WHITE (RX Computer)"
- note added: "low pass filter\nfcutoff = 159 Hz"
- note added: "may desire a voltage drop in \npass band too to measure \ninstantaneous currents \ngreater than 5A"
- note removed: "PIC32 schematic symbol. bring that in"
- note removed: "third prong???\n"
- moved on the sheet: J1, J2, J3, K1, R2, SW1

Commit message: revisions so far on final project page, mostly typos
Other:
- note added: "(RB13)"
Changed lines of the file:
@@
 Text Notes 1100 2900 0    197  ~ 0
 Outlet Box
-Text Notes 1750 4450 0    197  ~ 0
-PIC32 + Peripherals
-Text Notes 5300 5200 0    39   ~ 0
+Text Notes 5300 5200 0    47   ~ 0
 Inverter \n(Digital Output \n3.3V to 5V buffer)
 Text Notes 2300 950  0    39   ~ 0
@@
 	1950 5050 2300 5050
 Connection ~ 1950 5050
-Text Notes 1150 5400 0    39   ~ 0
+Text Notes 1150 5400 0    47   ~ 0
 low pass filter\nfcutoff = 159 Hz
-Text Notes 800  5750 0    39   ~ 0
+Text Notes 800  5850 0    47   ~ 0
 may desire a voltage drop in \npass band too to measure \ninstantaneous currents \ngreater than 5A
 Text Label 2300 4900 2    50   ~ 0
@@
 Wire Wire Line
 	1750 6400 1950 6400
-Text Notes 900  6200 0    39   ~ 0
+Text Notes 750  6200 0    47   ~ 0
 GREEN (TX Computer)\n
-Text Notes 900  6300 0    39   ~ 0
+Text Notes 750  6300 0    47   ~ 0
 WHITE (RX Computer)
-Text Notes 1300 6400 0    39   ~ 0
+Text Notes 750  6400 0    47   ~ 0
 BLACK
 Text Label 1950 6300 0    39   ~ 0
@@
 	1    0    0    -1
 $EndComp
-Text Notes 4200 4900 0    39   ~ 0
+Text Notes 4200 4900 0    47   ~ 0
 Indicator LEDs\n
 Wire Wire Line
@@
 Text Notes 3450 5900 0    39   ~ 0
 RA1
-Text Notes 3200 6000 0    39   ~ 0
+Text Notes 3150 6000 0    47   ~ 0
 (RB10)
-Text Notes 3200 5600 0    39   ~ 0
+Text Notes 3200 5600 0    47   ~ 0
 (RB0)
-Text Notes 3200 5800 0    39   ~ 0
+Text Notes 3200 5800 0    47   ~ 0
 (RB2)
-Text Notes 3200 5350 0    39   ~ 0
+Text Notes 3200 5350 0    47   ~ 0
 (RB1)
-Text Notes 3200 5150 0    39   ~ 0
+Text Notes 3200 5150 0    47   ~ 0
 (RA0)
+Text Notes 2500 5150 0    50   ~ 0
+(RB13)
+Text Notes 1750 4450 0    197  ~ 0
+PIC32 + Peripherals
 $EndSCHEMATC
