File: Schematic/_autosave-4760_Final.sch (KiCad schematic (older format))
At the start: 20 parts, among them J1 Supply (Input) Plug, J2 Client (Output) Sockets, J3 OutputPower, K1 G3NE-210T-US-DC5, Q1 AOT2618L NMOS, SW1 SW_SPST, U2 ACHS-7122

Commit message: revisions so far on final project page, mostly typos
Other:
- moved on the sheet: C3, D1, D2, D3, J?, Q1, R1, R2, R3, R4, R5, R6
